File: schematics/UV5R_full_EN/UV5R_full_EN.kicad_sch (KiCad schematic)
At the start: 22 parts, among them J1 TRS 2.5mm, J2 TS 3.5mm, Q1 2N2222, U1 PC817

Commit message: Correct schematic
Connections:
- net GPIO26: now also R9.1
Other:
- moved on the sheet: C1, C2, C5, D1, D2, J1, J2, R1, R10, R3, R5, R6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
