File: schematics/UV5R_full_ES/UV5R_full_ES.kicad_sch (KiCad schematic)
At the start: 22 parts, among them J1 TRS 2.5mm, J2 TS 3.5mm, Q1 2N2222, U1 PC817

Commit message: Correct schematic
Connections:
- net GPIO26: now also R9.1
Other:
- note added: "PTT opcion C — NPN sin aislar (requiere ACTIVE_HIGH=1)"
- note removed: "PTT opcion C — NPN pelado, sin aislar (requiere ACTIVE_HIGH=1)"
- title: Baofeng UV-5R -- interfaz funcional completa (plugs K1 de 2 pines) -> Baofeng UV-5R -- interfaz funcional completa 
- moved on the sheet: C4, C5, D1, D2, J1, J2, Q1, R10, R5, R6, R7, R9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
