File: schematics/APRS_Radio_Interface/APRS_Radio_Interface.kicad_pcb (KiCad board)
At the start: 2 copper layers, 0 parts

Commit message: Add APRS Coverage docs
Parts:
- added C1: 10uF, APRS_IF:CP_RAD_P2.54, F.Cu at (70.5, 30.0)
- added C2: 15nF, APRS_IF:C_DISC_P5.08, F.Cu at (50.0, 26.0)
- added C3: 15nF, APRS_IF:C_DISC_P5.08, F.Cu at (66.0, 26.0)
- added C4: 10uF, APRS_IF:CP_RAD_P2.54, F.Cu at (87.0, 55.0)
- added C5: 1nF, APRS_IF:C_DISC_P5.08, F.Cu at (60.0, 50.0)
- added D1: BAT54/1N4148, APRS_IF:D_DO35_P7.62, F.Cu at (54.0, 48.0)
- added D2: BAT54/1N4148, APRS_IF:D_DO35_P7.62, F.Cu at (46.0, 55.0)
- added D3: LED, APRS_IF:LED_P2.54, F.Cu at (88.0, 78.0)
- added D4: LED, APRS_IF:LED_P2.54, F.Cu at (66.0, 68.0)
- added J1: TRS 2.5mm, APRS_IF:HDR_1x03, F.Cu at (105.0, 42.0)
- added J2: TS 3.5mm, APRS_IF:HDR_1x02_13, F.Cu at (105.0, 62.0)
- added J3: ESP32, APRS_IF:HDR_1x05, F.Cu at (29.0, 50.0)
- added Q1: 2N2222, APRS_IF:TO92, F.Cu at (58.0, 72.0)
- added R1: 2k2, APRS_IF:R_AX_P10.16, F.Cu at (42.0, 30.0)
- added R10: 10k, APRS_IF:R_AX_P10.16, F.Cu at (58.0, 79.0)
- added R2: 2k2, APRS_IF:R_AX_P10.16, F.Cu at (58.0, 30.0)
- added R3: 10k, APRS_IF:R_AX_P10.16, F.Cu at (80.0, 30.0)
- added R5: 10k, APRS_IF:R_AX_P10.16, F.Cu at (82.0, 46.5)
- added R6: 10k, APRS_IF:R_AX_P10.16, F.Cu at (74.0, 61.0)
- added R7: 1k, APRS_IF:R_AX_P10.16, F.Cu at (76.0, 55.0)
- added R8: 220R, APRS_IF:R_AX_P10.16, F.Cu at (90.0, 72.0)
- added R9: 1k, APRS_IF:R_AX_P10.16, F.Cu at (76.0, 68.0)
- added RV1: 1k, APRS_IF:TRIM_3362P, F.Cu at (91.0, 31.0)
- added RV2: 10k, APRS_IF:TRIM_3362P, F.Cu at (96.0, 54.0)
- added U1: PC817, APRS_IF:DIP4, F.Cu at (101.0, 76.0)
Routing:
- net GND: track 0.00 -> 148.9 mm
- net SLEEVE (GND): track 0.00 -> 99.2 mm
- net +3V3: track 0.00 -> 94.7 mm
- net RING (PTT): track 0.00 -> 89.1 mm
- net GPIO26: track 0.00 -> 80.4 mm
- net GPIO33: track 0.00 -> 47.0 mm
- net SPKR: track 0.00 -> 32.1 mm
- net GPIO25: track 0.00 -> 18.1 mm
- net N$4: track 0.00 -> 17.5 mm
- net MIC: track 0.00 -> 16.8 mm
- net N$6: track 0.00 -> 15.1 mm
- net N$7: track 0.00 -> 14.4 mm
- net N$1: track 0.00 -> 7.77 mm
- net N$10: track 0.00 -> 7.23 mm
- net N$9: track 0.00 -> 6.85 mm
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Other:
- board outline added: 95 x 72 mm
- board text added: "+3V3"
- board text added: "Baofeng UV-5R interface - esp32_APRS_igate"
- board text added: "GND"
- board text added: "GPIO25 (TX audio)"
- board text added: "GPIO26 (PTT)"
- board text added: "GPIO33 (RX audio)"
- board text added: "J1 TRS 2.5mm"
- board text added: "J2 TS 3.5mm"
- board text added: "J3 -> ESP32"
- board text added: "PTT-A opto (isolated)"
- board text added: "PTT-C NPN (NOT isolated)"
- board text added: "RING = PTT"
- board text added: "SINGLE-SIDED: all copper on BOTTOM (B.Cu). Components on top."
- board text added: "SLV = GND-radio"
- board text added: "TIP = MIC"
- board text added: "TIP = SPKR"
- board text added: "TX audio ESP32 DAC -> radio MIC"
- board text added: "WIRE LINK (top): RV2.1 - J2.1"
